Commit message: base, standoff, holder

File: urdf/barista_robot_model.urdf (robot description, URDF)
Before this commit: robot barista, 0 links, 0 joints
Links:
- added link base_footprint
- added link base_link, mass 1.0; collision cylinder length=0.155 radius=0.178; visual cylinder length=0.155 radius=0.178
- added link cup_holder, mass 0.2; collision cylinder length=0.090 radius=0.160; visual cylinder length=0.090 radius=0.160
- added link standoff_rods, mass 0.02; collision cylinder length=0.220 radius=0.010; collision cylinder length=0.220 radius=0.010
Joints:
- added joint joint_base_footprint_base_link: type fixed, parent base_footprint, child base_link, origin xyz=0 0 0 rpy=0 0 0, axis 0 0 0
- added joint joint_base_link_standoff_rods: type fixed, parent base_link, child standoff_rods, origin xyz=0 0 0.1875 rpy=0 0 0, axis 0 0 0
- added joint joint_standoff_rods_cup_holder: type fixed, parent standoff_rods, child cup_holder, origin xyz=0 0 0.155 rpy=0 0 0, axis 0 0 0

Commit message: wheels and casters

File: urdf/barista_robot_model.urdf (robot description, URDF)
Before this commit: robot barista, 4 links, 3 joints
Links:
- added link back_pitch_link, mass 0.001; collision sphere radius=0.0325; visual sphere radius=0.0325
- added link back_roll_link, mass 0.001; collision cylinder length=0.001 radius=0.0045000000000000005; visual cylinder length=0.001 radius=0.0045000000000000005
- added link back_yaw_link, mass 0.001; collision cylinder length=0.001 radius=0.0045000000000000005; visual cylinder length=0.001 radius=0.0045000000000000005
- added link front_pitch_link, mass 0.001; collision sphere radius=0.0325; visual sphere radius=0.0325
- added link front_roll_link, mass 0.001; collision cylinder length=0.001 radius=0.0045000000000000005; visual cylinder length=0.001 radius=0.0045000000000000005
- added link front_yaw_link, mass 0.001; collision cylinder length=0.001 radius=0.0045000000000000005; visual cylinder length=0.001 radius=0.0045000000000000005
- added link left_wheel, mass 0.05; collision cylinder length=0.025 radius=0.04; visual cylinder length=0.025 radius=0.04
- added link right_wheel, mass 0.05; collision cylinder length=0.025 radius=0.04; visual cylinder length=0.025 radius=0.04
Joints:
- added joint back_pitch_joint: type continuous, parent back_roll_link, child back_pitch_link, origin xyz=0 0 0 rpy=0 0 0, axis 0 1 0, limit effort=1000.0 velocity=100.0
- added joint back_roll_joint: type continuous, parent back_yaw_link, child back_roll_link, origin xyz=0 0 0 rpy=0 0 0, axis 1 0 0, limit effort=1000.0 velocity=100.0
- added joint back_yaw_joint: type continuous, parent base_link, child back_yaw_link, origin xyz=-0.13 0 -0.0775 rpy=0 0 0, axis 0 0 1, limit effort=1000.0 velocity=100.0
- added joint front_pitch_joint: type continuous, parent front_roll_link, child front_pitch_link, origin xyz=0 0 0 rpy=0 0 0, axis 0 1 0, limit effort=1000.0 velocity=100.0
- added joint front_roll_joint: type continuous, parent front_yaw_link, child front_roll_link, origin xyz=0 0 0 rpy=0 0 0, axis 1 0 0, limit effort=1000.0 velocity=100.0
- added joint front_yaw_joint: type continuous, parent base_link, child front_yaw_link, origin xyz=0.13 0 -0.0775 rpy=0 0 0, axis 0 0 1, limit effort=1000.0 velocity=100.0
- added joint joint_base_link_left_wheel: type continuous, parent base_link, child left_wheel, origin xyz=0 0.145 -0.07 rpy=0 0 0, axis 0 1 0, limit effort=10000 velocity=1000
- added joint joint_base_link_right_wheel: type continuous, parent base_link, child right_wheel, origin xyz=0 -0.145 -0.07 rpy=0 0 0, axis 0 1 0, limit effort=10000 velocity=1000

Commit message: added laser scanner link to model

File: urdf/barista_robot_model.urdf (robot description, URDF)
Before this commit: robot barista, 12 links, 11 joints
Links:
- added link laser_scanner; collision mesh filename=package://barista_robot_description/meshes/hokuyo_urg_04lx.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 scale=1.0 1.0 1.0; visual mesh filename=package://barista_robot_description/meshes/hokuyo_urg_04lx.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 scale=1.0 1.0 1.0
Joints:
- added joint joint_base_link_laser_scanner: type fixed, parent base_link, child laser_scanner, origin xyz=0.13 0 0.0775 rpy=0 0 0, axis 0 0 0

Commit message: added plugins

File: urdf/barista_robot_model.urdf (robot description, URDF)
Before this commit: robot barista, 13 links, 12 joints
Links:
- link laser_scanner: mass None -> 0.160; geometry collision box size=0.050 0.050 0.070; visual mesh filename=package://barista_robot_description/meshes/hokuyo_urg_04lx.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 scale=1.0 1.0 1.0

Commit message: scanner position incorrect

File: urdf/barista_robot_model.urdf (robot description, URDF)
Before this commit: robot barista, 13 links, 12 joints
Links:
- added link laser_scan_frame
Joints:
- added joint laser_scan_frame_joint: type fixed, parent laser_scanner, child laser_scan_frame, origin xyz=0 0 0.03 rpy=0 0 0, axis 0 0 0

Commit message: illustrating scanner incorrect scanner rays pos

File: urdf/barista_robot_model.urdf (robot description, URDF)
Before this commit: robot barista, 14 links, 13 joints
Joints:
- joint laser_scan_frame_joint: origin xyz=0 0 0.03 rpy=0 0 0 -> xyz=0 0 1 rpy=0 0 0

Commit message: corrected incident points of laser rays in rviz2

File: urdf/barista_robot_model.urdf (robot description, URDF)
Before this commit: robot barista, 14 links, 13 joints
Joints:
- joint laser_scan_frame_joint: origin xyz=0 0 1 rpy=0 0 0 -> xyz=0 0 0.055 rpy=0 0 0

Commit message: mass & dimensions

File: urdf/barista_robot_model.urdf (robot description, URDF)
Before this commit: robot barista, 14 links, 13 joints
Links:
- removed link base_link
- added link chassis, mass 5.0; collision cylinder length=0.155 radius=0.178; visual cylinder length=0.155 radius=0.178
- link back_pitch_link: mass 0.001 -> 0.06; geometry collision sphere radius=0.0277; visual sphere radius=0.0277
- link cup_holder: mass 0.2 -> 1.0
- link front_pitch_link: mass 0.001 -> 0.06; geometry collision sphere radius=0.0277; visual sphere radius=0.0277
- link left_wheel: mass 0.05 -> 0.08; geometry collision cylinder length=0.0206 radius=0.0352; visual cylinder length=0.0206 radius=0.0352
- link right_wheel: mass 0.05 -> 0.08; geometry collision cylinder length=0.0206 radius=0.0352; visual cylinder length=0.0206 radius=0.0352
- link standoff_rods: mass 0.02 -> 0.4
Joints:
- removed joint joint_base_footprint_base_link
- removed joint joint_base_link_laser_scanner
- removed joint joint_base_link_left_wheel
- removed joint joint_base_link_right_wheel
- removed joint joint_base_link_standoff_rods
- added joint joint_base_footprint_chassis: type fixed, parent base_footprint, child chassis, origin xyz=0 0 0 rpy=0 0 0, axis 0 0 0
- added joint joint_chassis_laser_scanner: type fixed, parent chassis, child laser_scanner, origin xyz=0.13 0 0.0775 rpy=0 0 0, axis 0 0 0
- added joint joint_chassis_left_wheel: type continuous, parent chassis, child left_wheel, origin xyz=0 0.145 -0.07 rpy=0 0 0, axis 0 1 0, limit effort=10000 velocity=1000
- added joint joint_chassis_right_wheel: type continuous, parent chassis, child right_wheel, origin xyz=0 -0.145 -0.07 rpy=0 0 0, axis 0 1 0, limit effort=10000 velocity=1000
- added joint joint_chassis_standoff_rods: type fixed, parent chassis, child standoff_rods, origin xyz=0 0 0.1875 rpy=0 0 0, axis 0 0 0
- joint back_yaw_joint: parent base_link -> chassis
- joint front_yaw_joint: parent base_link -> chassis
