Commit message: xacro macros for standoffs and cup holder

File: xacro/barista_robot_model.urdf.xacro (robot description, xacro)
@@ -2,4 +2,6 @@
 <robot xmlns:xacro="http://www.ros.org/wiki/xacro" name="barista">
     <xacro:include filename="$(find barista_robot_description)/xacro/wheel.xacro"/>
+    <xacro:include filename="$(find barista_robot_description)/xacro/standoff.xacro"/>
+    <xacro:include filename="$(find barista_robot_description)/xacro/cup_holder_tray.xacro"/>
     <material name="blue">
         <color rgba="0.0 0.0 1.0 1.0"/>
@@ -42,58 +44,8 @@
     </joint>
     <link name="standoff_rods">
-        <visual>
-            <origin rpy="0 0 0" xyz="0.050 0.140 0"/>
-            <geometry>
-                <cylinder length="0.220" radius="0.010"/>
-            </geometry>
-            <material name="light_gray"/>
-        </visual>
-        <visual>
-            <origin rpy="0 0 0" xyz="-0.050 0.140 0"/>
-            <geometry>
-                <cylinder length="0.220" radius="0.010"/>
-            </geometry>
-            <material name="light_gray"/>
-        </visual>
-        <visual>
-            <origin rpy="0 0 0" xyz="0.050 -0.140 0"/>
-            <geometry>
-                <cylinder length="0.220" radius="0.010"/>
-            </geometry>
-            <material name="light_gray"/>
-        </visual>
-        <visual>
-            <origin rpy="0 0 0" xyz="-0.050 -0.140 0"/>
-            <geometry>
-                <cylinder length="0.220" radius="0.010"/>
-            </geometry>
-            <material name="light_gray"/>
-        </visual>
-        <!-- collision -->
-        <collision>
-            <origin rpy="0 0 0" xyz="0.050 0.140 0"/>
-            <geometry>
-                <cylinder length="0.220" radius="0.010"/>
-            </geometry>
-        </collision>
-        <collision>
-            <origin rpy="0 0 0" xyz="-0.050 0.140 0"/>
-            <geometry>
-                <cylinder length="0.220" radius="0.010"/>
-            </geometry>
-        </collision>
-        <collision>
-            <origin rpy="0 0 0" xyz="0.050 -0.140 0"/>
-            <geometry>
-                <cylinder length="0.220" radius="0.010"/>
-            </geometry>
-        </collision>
-        <collision>
-            <origin rpy="0 0 0" xyz="-0.050 -0.140 0"/>
-            <geometry>
-                <cylinder length="0.220" radius="0.010"/>
-            </geometry>
-            <material name="light_gray"/>
-        </collision>
+        <xacro:standoff x_coord="0.050" y_coord="0.140"/>
+        <xacro:standoff x_coord="-0.050" y_coord="0.140"/>
+        <xacro:standoff x_coord="0.050" y_coord="-0.140"/>
+        <xacro:standoff x_coord="-0.050" y_coord="-0.140"/>
         <!-- approximate a very light box with size [0.1, 0.28, 0.22] -->
         <inertial>
@@ -109,24 +61,5 @@
         <axis xyz="0 0 0"/>
     </joint>
-    <link name="cup_holder">
-        <visual>
-            <origin rpy="0 0 0" xyz="0 0 0"/>
-            <geometry>
-                <cylinder length="0.090" radius="0.160"/>
-            </geometry>
-            <material name="blue"/>
-        </visual>
-        <collision>
-            <origin rpy="0 0 0" xyz="0 0 0"/>
-            <geometry>
-                <cylinder length="0.090" radius="0.160"/>
-            </geometry>
-        </collision>
-        <inertial>
-            <mass value="1.0"/>
-            <origin rpy="0 0 0" xyz="0 0 0"/>
-            <inertia ixx="0.007075" ixy="0.0" ixz="0.0" iyy="0.007075" iyz="0.0" izz="0.0128"/>
-        </inertial>
-    </link>
+    <xacro:cup_holder_tray/>
     <gazebo reference="cup_holder">
         <material>Gazebo/Blue</material>

Commit message: unconditional laser scanner

File: xacro/barista_robot_model.urdf.xacro (robot description, xacro)
@@ -4,4 +4,5 @@
     <xacro:include filename="$(find barista_robot_description)/xacro/standoff.xacro"/>
     <xacro:include filename="$(find barista_robot_description)/xacro/cup_holder_tray.xacro"/>
+    <xacro:include filename="$(find barista_robot_description)/xacro/laser_scanner.xacro"/>
     <material name="blue">
         <color rgba="0.0 0.0 1.0 1.0"/>
@@ -304,10 +305,9 @@
   </joint>
    <!-- Laser scanner -->
-   <link name="laser_scanner">
+   <!-- <link name="laser_scanner">
         <visual>
             <origin rpy="0 0 0" xyz="0 0 0"/>
             <geometry>
                 <mesh filename="package://barista_robot_description/meshes/hokuyo_urg_04lx.stl" scale="1.0 1.0 1.0"/>
-                <!-- <mesh filename="package://box_bot_description/meshes/hokuyo_urg_04lx.stl" scale="1.0 1.0 1.0"/> -->
             </geometry>
             <material name="light_gray"/>
@@ -317,5 +317,4 @@
             <geometry>
                 <box size="0.050 0.050 0.070"/>
-                <!-- <mesh filename="package://barista_robot_description/meshes/hokuyo_urg_04lx.stl" scale="1.0 1.0 1.0"/> -->
             </geometry>
         </collision>
@@ -339,5 +338,5 @@
         <child link="laser_scan_frame"/>
         <axis xyz="0 0 0"/>
-    </joint>
+    </joint> -->
    <!-- Plugins -->
    <!-- Joint publisher (for Gazebo)-->
@@ -379,5 +378,5 @@
    <!-- Sensors (with plugins) -->
   <!-- Laser scanner (simulated) -->
-  <gazebo reference="laser_scan_frame">
+  <!-- <gazebo reference="laser_scan_frame">
     <sensor name="sensor_ray" type="ray">
       <pose>0 0 0 0 0 0</pose>
@@ -393,5 +392,4 @@
         <range>
           <min>0.1</min>
-          <!-- <min>0.4</min> -->
           <max>5.0</max>
         </range>
@@ -399,6 +397,5 @@
       <always_on>true</always_on>
       <visualize>true</visualize>
-      <!-- <update_rate>100.0</update_rate> -->
-      <update_rate>10.0</update_rate> <!-- 10, 15, 20, 30 Hz -->
+      <update_rate>10.0</update_rate>
       <plugin name="laser" filename="libgazebo_ros_ray_sensor.so">
         <ros>
@@ -410,4 +407,5 @@
       </plugin>
     </sensor>
-  </gazebo>
+  </gazebo> -->
+  <xacro:laser_scanner/>
 </robot>

Commit message: part 2 submission notes

File: xacro/barista_robot_model.urdf.xacro (robot description, xacro)
@@ -4,5 +4,5 @@
     <xacro:include filename="$(find barista_robot_description)/xacro/standoff.xacro"/>
     <xacro:include filename="$(find barista_robot_description)/xacro/cup_holder_tray.xacro"/>
-    <xacro:arg name="include_scanner" default="true"/>
+    <xacro:arg name="include_laser" default="true"/>
     <material name="blue">
         <color rgba="0.0 0.0 1.0 1.0"/>
@@ -304,39 +304,4 @@
     <dynamics damping="0.0" friction="0.1"/>
   </joint>
-   <!-- Laser scanner -->
-   <!-- <link name="laser_scanner">
-        <visual>
-            <origin rpy="0 0 0" xyz="0 0 0"/>
-            <geometry>
-                <mesh filename="package://barista_robot_description/meshes/hokuyo_urg_04lx.stl" scale="1.0 1.0 1.0"/>
-            </geometry>
-            <material name="light_gray"/>
-        </visual>
-        <collision>
-            <origin rpy="0 0 0" xyz="0 0 0"/>
-            <geometry>
-                <box size="0.050 0.050 0.070"/>
-            </geometry>
-        </collision>
-        <inertial>
-            <mass value="0.160"/>
-            <origin rpy="0 0 0" xyz="0 0 0"/>
-            <inertia ixx="9.866666666666669e-05" ixy="0.0" ixz="0.0" iyy="9.866666666666669e-05" iyz="0.0" izz="6.666666666666668e-05"/>
-        </inertial>
-    </link>
-    <joint name="joint_chassis_laser_scanner" type="fixed">
-        <origin rpy="0 0 0" xyz="0.13 0 0.0775"/>
-        <parent link="chassis"/>
-        <child link="laser_scanner"/>
-        <axis xyz="0 0 0"/>
-    </joint>
-    <link name="laser_scan_frame">
-    </link>
-    <joint name="laser_scan_frame_joint" type="fixed">
-        <origin rpy="0 0 0" xyz="0 0 0.055"/>
-        <parent link="laser_scanner"/>
-        <child link="laser_scan_frame"/>
-        <axis xyz="0 0 0"/>
-    </joint> -->
    <!-- Plugins -->
    <!-- Joint publisher (for Gazebo)-->
@@ -377,5 +342,5 @@
   </gazebo>
   <!-- Laser scanner (conditional) -->
-    <xacro:if value="$(arg include_scanner)">
+    <xacro:if value="$(arg include_laser)">
         <xacro:include filename="$(find barista_robot_description)/xacro/laser_scanner.xacro"/>
         <xacro:laser_scanner/>

Commit message: first attempt to spawn two robots
1. Gazebo took some time but showed both bots.
2. Rviz2 has to be configured and errors removed.

File: xacro/barista_robot_model.urdf.xacro (robot description, xacro)
@@ -1,8 +1,8 @@
 <?xml version="1.6"?>
 <robot xmlns:xacro="http://www.ros.org/wiki/xacro" name="barista">
+    <xacro:property name="robot_name" value="$(arg robot_name)"/>
     <xacro:include filename="$(find barista_robot_description)/xacro/wheel.xacro"/>
     <xacro:include filename="$(find barista_robot_description)/xacro/standoff.xacro"/>
     <xacro:include filename="$(find barista_robot_description)/xacro/cup_holder_tray.xacro"/>
-    <xacro:arg name="include_laser" default="true"/>
     <material name="blue">
         <color rgba="0.0 0.0 1.0 1.0"/>
@@ -309,4 +309,5 @@
     <plugin name="bar_bot_joint_state" filename="libgazebo_ros_joint_state_publisher.so">
       <ros>
+          <namespace>/${robot_name}</namespace>
           <remapping>~/out:=joint_states</remapping>
       </ros>
@@ -325,4 +326,9 @@
    <gazebo>
     <plugin filename="libgazebo_ros_diff_drive.so" name="differential_drive_controller">
+      <!-- namespace for multiple robots from the same model-->
+      <ros>
+        <namespace>/${robot_name}</namespace>
+        <remapping>/cmd_vel:=cmd_vel</remapping>
+      </ros>
       <!-- wheels -->
       <left_joint>joint_chassis_left_wheel</left_joint>
@@ -337,9 +343,10 @@
       <publish_odom>true</publish_odom>
       <publish_odom_tf>true</publish_odom_tf>
-      <odometry_frame>odom</odometry_frame>
-      <robot_base_frame>base_footprint</robot_base_frame>
+      <odometry_frame>${robot_name}/odom</odometry_frame>
+      <robot_base_frame>${robot_name}/base_footprint</robot_base_frame>
     </plugin>
   </gazebo>
   <!-- Laser scanner (conditional) -->
+    <xacro:arg name="include_laser" default="true"/>
     <xacro:if value="$(arg include_laser)">
         <xacro:include filename="$(find barista_robot_description)/xacro/laser_scanner.xacro"/>

File: xacro/laser_scanner.xacro (robot description, xacro)
@@ -60,5 +60,6 @@
       <plugin name="laser" filename="libgazebo_ros_ray_sensor.so">
         <ros>
-          <!-- <namespace>/bar_bot</namespace> -->
+          <!-- Expect xacro:property robot_name-->
+          <namespace>/${robot_name}</namespace>
           <remapping>~/out:=/scan</remapping>
         </ros>

Commit message: different colors

File: xacro/barista_robot_model.urdf.xacro (robot description, xacro)
@@ -14,4 +14,12 @@
         <color rgba="0.0 0.0 0.0 1.0"/>
     </material>
+    <xacro:if value="${robot_name == 'morty'}">
+        <xacro:property name="base_color_rviz" value="blue"/>
+        <xacro:property name="base_color_gazebo" value="Gazebo/Blue"/>
+    </xacro:if>
+    <xacro:unless value="${robot_name == 'morty'}">
+        <xacro:property name="base_color_rviz" value="red"/>
+        <xacro:property name="base_color_gazebo" value="Gazebo/Red"/>
+    </xacro:unless>
     <!-- Robot base/root link -->
     <link name="base_footprint"/>
@@ -22,6 +30,6 @@
                 <cylinder length="0.155" radius="0.178"/>
             </geometry>
-            <material name="blue"/>
-        </visual>
+            <material name="${base_color_rviz}"/>
+       </visual>
         <collision>
             <origin rpy="0 0 0" xyz="0 0 0"/>
@@ -37,5 +45,5 @@
     </link>
     <gazebo reference="chassis">
-        <material>Gazebo/Blue</material>
+        <material>${base_color_gazebo}</material>
     </gazebo>
     <joint name="joint_base_footprint_chassis" type="fixed">
@@ -65,5 +73,5 @@
     <xacro:cup_holder_tray/>
     <gazebo reference="cup_holder">
-        <material>Gazebo/Blue</material>
+        <material>${base_color_gazebo}</material>
     </gazebo>
     <joint name="joint_standoff_rods_cup_holder" type="fixed">

File: xacro/cup_holder_tray.xacro (robot description, xacro)
@@ -10,5 +10,5 @@
                     <cylinder length="${cup_holder_length}" radius="${cup_holder_radius}"/>
                 </geometry>
-                <material name="blue"/>
+                <material name="${base_color_rviz}"/>
             </visual>
             <collision>
